File: DrillBoard-Hardware.sch (KiCad schematic (older format))
At the start: 29 parts

Commit message: General layout done, routing is a work in progress.
Parts:
- removed U?: TM4C129E_Launchpad_JTAG_Side, symbol TM4C129E_Launchpad_JTAG_Side
- added U6: TM4C129E_Launchpad_X9, MRDT-Shields:TM4C129E_Launchpad_X9, symbol TM4C129E_Launchpad_X9
- 10u1, 10u2: renamed from 10u; footprint (none) -> Capacitors_SMD:C_0805_HandSoldering
- C1, C2: renamed from C?; footprint (none) -> MRDT-Connectors:Anderson_3_Horisontal_Side-by-Side
- C10, C11, C3, C4, C9: renamed from C?; footprint (none) -> Capacitors_SMD:C_0805_HandSoldering
- C7, C8: renamed from C?; footprint (none) -> MRDT-Connectors:Anderson_2_Side-by-Side
- R1, R2, R3, R4, R5, R6: renamed from R?; footprint (none) -> Resistors_SMD:R_0805_HandSoldering
- U1, U2: renamed from U?; footprint (none) -> MRDT-ICs:MultiPowerSO-30
- U3: renamed from U?; footprint (none) -> MRDT-Devices:OKI
- U4: renamed from U?; footprint (none) -> Housings_SOIC:SOIC-16_3.9x9.9mm_Pitch1.27mm
- U5: renamed from U?; footprint (none) -> MRDT-Connectors:MOLEX_SL_5
- U7, U8: renamed from U?; footprint (none) -> MRDT-connectors:MOLEX_SL_3
- gave numbers to parts that had none: 4
Changed lines of the file:
@@
 $EndDescr
 $Comp
-L VNH5019A-E U?
+L VNH5019A-E U2
 U 1 1 5AA58283
 P 2550 7200
-F 0 "U?" H 2600 5850 60  0000 C CNN
+F 0 "U2" H 2600 5850 60  0000 C CNN
 F 1 "VNH5019A-E" H 3150 8650 60  0000 C CNN
-F 2 "" H 2550 7200 60  0001 C CNN
+F 2 "MRDT-ICs:MultiPowerSO-30" H 2550 7200 60  0001 C CNN
 F 3 "" H 2550 7200 60  0001 C CNN
 	1    2550 7200
@@
 $EndComp
 $Comp
-L VNH5019A-E U?
+L VNH5019A-E U1
 U 1 1 5AA582EF
 P 2550 5100
-F 0 "U?" H 2600 2950 60  0000 C CNN
+F 0 "U1" H 2600 2950 60  0000 C CNN
 F 1 "VNH5019A-E" H 3150 6550 60  0000 C CNN
-F 2 "" H 2550 5100 60  0001 C CNN
+F 2 "MRDT-ICs:MultiPowerSO-30" H 2550 5100 60  0001 C CNN
 F 3 "" H 2550 5100 60  0001 C CNN
 	1    2550 5100
@@
 GND
 $Comp
-L Anderson-2 C?
+L Anderson-2 C7
 U 1 1 5AA58F86
 P 4450 4200
-F 0 "C?" H 4500 4150 60  0000 C CNN
+F 0 "C7" H 4500 4150 60  0000 C CNN
 F 1 "Anderson-2" H 4550 4700 60  0000 C CNN
-F 2 "" H 4500 3650 60  0001 C CNN
+F 2 "MRDT-Connectors:Anderson_2_Side-by-Side" H 4500 3650 60  0001 C CNN
 F 3 "" H 4500 3650 60  0001 C CNN
 	1    4450 4200
@@
 $EndComp
 $Comp
-L Anderson-2 C?
+L Anderson-2 C8
 U 1 1 5AA59025
 P 4450 6300
-F 0 "C?" H 4500 6250 60  0000 C CNN
+F 0 "C8" H 4500 6250 60  0000 C CNN
 F 1 "Anderson-2" H 4550 6800 60  0000 C CNN
-F 2 "" H 4500 5750 60  0001 C CNN
+F 2 "MRDT-Connectors:Anderson_2_Side-by-Side" H 4500 5750 60  0001 C CNN
 F 3 "" H 4500 5750 60  0001 C CNN
 	1    4450 6300
@@
 Text Notes 4300 5700 0    60   ~ 0
 Motor 2
-$Comp
-L TM4C129E_Launchpad_JTAG_Side U?
-U 1 1 5AA59663
-P 9100 4200
-F 0 "U?" H 9200 4150 60  0001 C CNN
-F 1 "TM4C129E_Launchpad_JTAG_Side" H 9350 6600 60  0000 C CNN
-F 2 "" H 9250 8200 60  0001 C CNN
-F 3 "" H 9250 8200 60  0001 C CNN
-	1    9100 4200
-	1    0    0    -1
-$EndComp
 Text GLabel 8900 3750 0    60   Input ~ 0
 PWM2
@@
 PWM2
 $Comp
-L OKI U?
+L OKI U3
 U 1 1 5AA5A472
 P 2700 2600
-F 0 "U?" H 2550 2350 60  0001 C CNN
+F 0 "U3" H 2550 2350 60  0001 C CNN
 F 1 "OKI" H 2850 2950 60  0000 C CNN
-F 2 "" H 2450 2500 60  0001 C CNN
+F 2 "MRDT-Devices:OKI" H 2450 2500 60  0001 C CNN
 F 3 "" H 2450 2500 60  0001 C CNN
 	1    2700 2600
@@
 $EndComp
 $Comp
-L C 10u
+L C 10u1
 U 1 1 5AA5A5BB
 P 2250 2350
-F 0 "10u" V 2100 2300 50  0000 L CNN
+F 0 "10u1" V 2100 2300 50  0000 L CNN
 F 1 "C" H 2275 2250 50  0000 L CNN
-F 2 "" H 2288 2200 50  0001 C CNN
+F 2 "Capacitors_SMD:C_0805_HandSoldering" H 2288 2200 50  0001 C CNN
 F 3 "" H 2250 2350 50  0001 C CNN
 	1    2250 2350
@@
 $EndComp
 $Comp
-L C 10u
+L C 10u2
 U 1 1 5AA5A657
 P 2250 2550
-F 0 "10u" V 2400 2500 50  0000 L CNN
+F 0 "10u2" V 2400 2500 50  0000 L CNN
 F 1 "C" H 2275 2450 50  0000 L CNN
-F 2 "" H 2288 2400 50  0001 C CNN
+F 2 "Capacitors_SMD:C_0805_HandSoldering" H 2288 2400 50  0001 C CNN
 F 3 "" H 2250 2550 50  0001 C CNN
 	1    2250 2550
@@
 +3V3
 $Comp
-L Anderson-3 C?
+L Anderson-3 C1
 U 1 1 5AA5A2E6
 P 2700 1900
-F 0 "C?" H 2750 1850 60  0000 C CNN
+F 0 "C1" H 2750 1850 60  0000 C CNN
 F 1 "Anderson-3" H 2850 2650 60  0000 C CNN
-F 2 "" H 2750 1350 60  0001 C CNN
+F 2 "MRDT-Connectors:Anderson_3_Horisontal_Side-by-Side" H 2750 1350 60  0001 C CNN
 F 3 "" H 2750 1350 60  0001 C CNN
 	1    2700 1900
@@
 +12V
 $Comp
-L Fuse F?
+L Fuse F1
 U 1 1 5AA5CCC9
 P 2200 1500
-F 0 "F?" V 2280 1500 50  0000 C CNN
+F 0 "F1" V 2280 1500 50  0000 C CNN
 F 1 "Fuse-2A" V 2100 1450 50  0000 C CNN
 F 2 "" V 2130 1500 50  0001 C CNN
@@
 $EndComp
 $Comp
-L Anderson-3 C?
+L Anderson-3 C2
 U 1 1 5AA5CF97
 P 3500 1900
-F 0 "C?" H 3550 1850 60  0000 C CNN
+F 0 "C2" H 3550 1850 60  0000 C CNN
 F 1 "Anderson-3" H 3650 2650 60  0000 C CNN
-F 2 "" H 3550 1350 60  0001 C CNN
+F 2 "MRDT-Connectors:Anderson_3_Horisontal_Side-by-Side" H 3550 1350 60  0001 C CNN
 F 3 "" H 3550 1350 60  0001 C CNN
 	1    3500 1900
@@
 Right Side
 $Comp
-L 3P1T_Fused SW?
+L 3P1T_Fused SW1
 U 1 1 5AA5E3EE
 P 6250 3500
-F 0 "SW?" H 6350 3450 60  0000 C CNN
+F 0 "SW1" H 6350 3450 60  0000 C CNN
 F 1 "3P1T_Fused" H 6650 4100 60  0000 C CNN
 F 2 "" H 6250 3500 60  0001 C CNN
@@
 	4350 5900 3950 5900
 $Comp
-L R R?
+L R R2
 U 1 1 5AA63460
 P 2200 4650
-F 0 "R?" V 2280 4650 50  0000 C CNN
+F 0 "R2" V 2280 4650 50  0000 C CNN
 F 1 "1K" V 2200 4650 50  0000 C CNN
-F 2 "" V 2130 4650 50  0001 C CNN
+F 2 "Resistors_SMD:R_0805_HandSoldering" V 2130 4650 50  0001 C CNN
 F 3 "" H 2200 4650 50  0001 C CNN
 	1    2200 4650
@@
 $EndComp
 $Comp
-L R R?
+L R R5
 U 1 1 5AA63587
 P 2200 6750
-F 0 "R?" V 2280 6750 50  0000 C CNN
+F 0 "R5" V 2280 6750 50  0000 C CNN
 F 1 "1K" V 2200 6750 50  0000 C CNN
-F 2 "" V 2130 6750 50  0001 C CNN
+F 2 "Resistors_SMD:R_0805_HandSoldering" V 2130 6750 50  0001 C CNN
 F 3 "" H 2200 6750 50  0001 C CNN
 	1    2200 6750
@@
 $EndComp
 $Comp
-L R R?
+L R R4
 U 1 1 5AA63773
 P 2200 6450
-F 0 "R?" V 2100 6450 50  0000 C CNN
+F 0 "R4" V 2100 6450 50  0000 C CNN
 F 1 "1K" V 2200 6450 50  0000 C CNN
-F 2 "" V 2130 6450 50  0001 C CNN
+F 2 "Resistors_SMD:R_0805_HandSoldering" V 2130 6450 50  0001 C CNN
 F 3 "" H 2200 6450 50  0001 C CNN
 	1    2200 6450
@@
 $EndComp
 $Comp
-L R R?
+L R R6
 U 1 1 5AA637B2
 P 2200 7050
-F 0 "R?" V 2280 7050 50  0000 C CNN
+F 0 "R6" V 2280 7050 50  0000 C CNN
 F 1 "1K" V 2200 7050 50  0000 C CNN
-F 2 "" V 2130 7050 50  0001 C CNN
+F 2 "Resistors_SMD:R_0805_HandSoldering" V 2130 7050 50  0001 C CNN
 F 3 "" H 2200 7050 50  0001 C CNN
 	1    2200 7050
@@
 $EndComp
 $Comp
-L R R?
+L R R3
 U 1 1 5AA63832
 P 2200 4950
-F 0 "R?" V 2280 4950 50  0000 C CNN
+F 0 "R3" V 2280 4950 50  0000 C CNN
 F 1 "1K" V 2200 4950 50  0000 C CNN
-F 2 "" V 2130 4950 50  0001 C CNN
+F 2 "Resistors_SMD:R_0805_HandSoldering" V 2130 4950 50  0001 C CNN
 F 3 "" H 2200 4950 50  0001 C CNN
 	1    2200 4950
@@
 $EndComp
 $Comp
-L R R?
+L R R1
 U 1 1 5AA639F0
 P 2200 4350
-F 0 "R?" V 2100 4350 50  0000 C CNN
+F 0 "R1" V 2100 4350 50  0000 C CNN
 F 1 "1K" V 2200 4350 50  0000 C CNN
-F 2 "" V 2130 4350 50  0001 C CNN
+F 2 "Resistors_SMD:R_0805_HandSoldering" V 2130 4350 50  0001 C CNN
 F 3 "" H 2200 4350 50  0001 C CNN
 	1    2200 4350
@@
 PL5-PM2
 $Comp
-L C C?
+L C C11
 U 1 1 5AA665A9
 P 7500 5150
-F 0 "C?" H 7525 5250 50  0000 L CNN
+F 0 "C11" H 7525 5250 50  0000 L CNN
 F 1 "1u" H 7525 5050 50  0000 L CNN
-F 2 "" H 7538 5000 50  0001 C CNN
+F 2 "Capacitors_SMD:C_0805_HandSoldering" H 7538 5000 50  0001 C CNN
 F 3 "" H 7500 5150 50  0001 C CNN
 	1    7500 5150
@@
 $EndComp
 $Comp
-L C C?
+L C C4
 U 1 1 5AA66688
 P 4150 6850
-F 0 "C?" H 4175 6950 50  0000 L CNN
+F 0 "C4" H 4175 6950 50  0000 L CNN
 F 1 ".1u" H 4175 6750 50  0000 L CNN
-F 2 "" H 4188 6700 50  0001 C CNN
+F 2 "Capacitors_SMD:C_0805_HandSoldering" H 4188 6700 50  0001 C CNN
 F 3 "" H 4150 6850 50  0001 C CNN
 	1    4150 6850
@@
 GND
 $Comp
-L CP1 C?
+L CP1 C5
 U 1 1 5AA670E6
 P 4400 4750
-F 0 "C?" H 4425 4850 50  0000 L CNN
+F 0 "C5" H 4425 4850 50  0000 L CNN
 F 1 "47u" H 4425 4650 50  0000 L CNN
 F 2 "" H 4400 4750 50  0001 C CNN
@@
 $EndComp
 $Comp
-L CP1 C?
+L CP1 C6
 U 1 1 5AA671B2
 P 4400 6850
-F 0 "C?" H 4425 6950 50  0000 L CNN
+F 0 "C6" H 4425 6950 50  0000 L CNN
 F 1 "47u" H 4425 6750 50  0000 L CNN
 F 2 "" H 4400 6850 50  0001 C CNN
@@
 $EndComp
 $Comp
-L Molex_SL-3 U?
+L Molex_SL-3 U7
 U 1 1 5AA67B2B
 P 9700 4900
-F 0 "U?" H 9750 4850 60  0001 C CNN
+F 0 "U7" H 9750 4850 60  0001 C CNN
 F 1 "Molex_SL-3" H 9750 5250 60  0000 C CNN
-F 2 "" H 9700 4900 60  0001 C CNN
+F 2 "MRDT-connectors:MOLEX_SL_3" H 9700 4900 60  0001 C CNN
 F 3 "" H 9700 4900 60  0001 C CNN
 	1    9700 4900
@@
 $EndComp
 $Comp
-L Molex_SL-3 U?
+L Molex_SL-3 U8
 U 1 1 5AA67B79
 P 9700 5350
-F 0 "U?" H 9750 5300 60  0001 C CNN
+F 0 "U8" H 9750 5300 60  0001 C CNN
 F 1 "Molex_SL-3" H 9750 5700 60  0000 C CNN
-F 2 "" H 9700 5350 60  0001 C CNN
+F 2 "MRDT-connectors:MOLEX_SL_3" H 9700 5350 60  0001 C CNN
 F 3 "" H 9700 5350 60  0001 C CNN
 	1    9700 5350
@@
 Encoder2_PWM
 $Comp
-L Molex_SL-5 U?
+L Molex_SL-5 U5
 U 1 1 5AA68D20
 P 7800 6250
-F 0 "U?" H 7850 6200 60  0001 C CNN
+F 0 "U5" H 7850 6200 60  0001 C CNN
 F 1 "Molex_SL-5" H 8000 6800 60  0000 C CNN
-F 2 "" H 7800 6250 60  0001 C CNN
+F 2 "MRDT-Connectors:MOLEX_SL_5" H 7800 6250 60  0001 C CNN
 F 3 "" H 7800 6250 60  0001 C CNN
 	1    7800 6250
@@
 Serial (7/6)
 $Comp
-L MAX-3232 U?
+L MAX-3232 U4
 U 1 1 5AA6A21C
 P 6550 5950
-F 0 "U?" H 6600 5900 60  0000 C CNN
+F 0 "U4" H 6600 5900 60  0000 C CNN
 F 1 "MAX-3232" H 6850 6800 60  0000 C CNN
-F 2 "" H 6550 5300 60  0001 C CNN
+F 2 "Housings_SOIC:SOIC-16_3.9x9.9mm_Pitch1.27mm" H 6550 5300 60  0001 C CNN
 F 3 "" H 6550 5300 60  0001 C CNN
 	1    6550 5950
@@
 +3V3
 $Comp
-L C C?
+L C C9
 U 1 1 5AA6AB65
 P 6200 5050
-F 0 "C?" H 6225 5150 50  0000 L CNN
+F 0 "C9" H 6225 5150 50  0000 L CNN
 F 1 "1u" H 6225 4950 50  0000 L CNN
-F 2 "" H 6238 4900 50  0001 C CNN
+F 2 "Capacitors_SMD:C_0805_HandSoldering" H 6238 4900 50  0001 C CNN
 F 3 "" H 6200 5050 50  0001 C CNN
 	1    6200 5050
@@
 $EndComp
 $Comp
-L C C?
+L C C10
 U 1 1 5AA6ABC5
 P 6200 5400
-F 0 "C?" H 6225 5500 50  0000 L CNN
+F 0 "C10" H 6225 5500 50  0000 L CNN
 F 1 "1u" H 6225 5300 50  0000 L CNN
-F 2 "" H 6238 5250 50  0001 C CNN
+F 2 "Capacitors_SMD:C_0805_HandSoldering" H 6238 5250 50  0001 C CNN
 F 3 "" H 6200 5400 50  0001 C CNN
 	1    6200 5400
@@
 $EndComp
 $Comp
-L C C?
+L C C3
 U 1 1 5AA6AC26
 P 4150 4750
-F 0 "C?" H 4175 4850 50  0000 L CNN
+F 0 "C3" H 4175 4850 50  0000 L CNN
 F 1 ".1u" H 4175 4650 50  0000 L CNN
-F 2 "" H 4188 4600 50  0001 C CNN
+F 2 "Capacitors_SMD:C_0805_HandSoldering" H 4188 4600 50  0001 C CNN
 F 3 "" H 4150 4750 50  0001 C CNN
 	1    4150 4750
@@
 Text GLabel 6350 5800 0    60   Output ~ 0
 RX
+$Comp
+L TM4C129E_Launchpad_X9 U6
+U 1 1 5AA5C9A5
+P 9100 4200
+F 0 "U6" H 9200 4150 60  0001 C CNN
+F 1 "TM4C129E_Launchpad_X9" H 9350 6600 60  0000 C CNN
+F 2 "MRDT-Shields:TM4C129E_Launchpad_X9" H 9250 8200 60  0001 C CNN
+F 3 "" H 9250 8200 60  0001 C CNN
+	1    9100 4200
+	1    0    0    -1
+$EndComp
 $EndSCHEMATC

Commit message: Created board layout
Will run traces this wek in preparation for board review next Sunday.
Parts:
- removed C2: Anderson-3, MRDT-Connectors:Anderson_3_Horisontal_Side-by-Side, symbol Anderson-3
- removed C3: .1u, Capacitors_SMD:C_0805_HandSoldering, symbol C
- removed C5: 47u, symbol CP1
- removed F1: Fuse-2A, symbol Fuse
- added C13, C14: 1u, Capacitors_SMD:C_0603_HandSoldering, symbol C
- C1: footprint MRDT-Connectors:Anderson_3_Horisontal_Side-by-Side -> MRDT_Connectors:Anderson_3_Horisontal_Side_by_Side
- C10, C11, C4, C9: footprint Capacitors_SMD:C_0805_HandSoldering -> Capacitors_SMD:C_0603_HandSoldering
- C12: renamed from 10u2; value C -> 10u; footprint Capacitors_SMD:C_0805_HandSoldering -> Capacitors_SMD:C_0603_HandSoldering
- C2: renamed from 10u1; value C -> 10u; footprint Capacitors_SMD:C_0805_HandSoldering -> Capacitors_SMD:C_0603_HandSoldering
- C6: footprint (none) -> Capacitors_THT:CP_Radial_D5.0mm_P2.50mm
- C7, C8: footprint MRDT-Connectors:Anderson_2_Side-by-Side -> MRDT_Connectors:Anderson_2_Horisontal_Side_by_Side
- R1, R2, R3, R4, R5, R6: footprint Resistors_SMD:R_0805_HandSoldering -> Resistors_SMD:R_0603_HandSoldering
- SW1: footprint (none) -> MRDT_Switches:3P1T_Switch
- U1, U2: footprint MRDT-ICs:MultiPowerSO-30 -> MRDT_ICs:MultiPowerSO_30
- U3: footprint MRDT-Devices:OKI -> MRDT_Devices:OKI_Horisontal
- U5: footprint MRDT-Connectors:MOLEX_SL_5 -> MRDT_Connectors:MOLEX_SL_5
- U6: footprint MRDT-Shields:TM4C129E_Launchpad_X9 -> MRDT_Shields:TM4C129E_Launchpad_X9
- U7, U8: value Molex_SL-3 -> Picoblade-3; footprint MRDT-connectors:MOLEX_SL_3 -> Connectors_Molex:Molex_PicoBlade_53047-0310_03x1.25mm_Straight; symbol Molex_SL-3 -> Picoblade_3
Connections:
- net labels added: 12V_Logic, Out_A1, Out_A2, Out_B1, Out_B2
- wire segments 48 -> 53
Other:
- note added: "Encoders"
- note added: "Power"
- note added: "Serial"
- note removed: "Left Side"
- note removed: "Right Side"
- moved on the sheet: C4, C6
