File: _saved_DrillBoard-Hardware.sch (KiCad schematic (older format))
At the start: 31 parts, among them SW1 3P1T_Fused, U1 VNH5019A-E, U10 LS_4, U2 VNH5019A-E, U3 OKI, U4 LS_1, U5 LS_2, U6 TM4C129E_Launchpad_X9, U7 Picoblade-3, U8 Picoblade-3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

Commit message: Finalized schematic and board and generated Gerbs
Parts:
- U7, U8: footprint Connectors_Molex:Molex_PicoBlade_53047-0310_03x1.25mm_Straight -> MRDT_Connectors:MOLEX_SL_3_Vertical
Changed lines of the file:
@@
 F 0 "U7" H 9750 4850 60  0001 C CNN
 F 1 "Picoblade-3" H 9750 5250 60  0000 C CNN
-F 2 "Connectors_Molex:Molex_PicoBlade_53047-0310_03x1.25mm_Straight" H 9700 4900 60  0001 C CNN
+F 2 "MRDT_Connectors:MOLEX_SL_3_Vertical" H 9700 4900 60  0001 C CNN
 F 3 "" H 9700 4900 60  0001 C CNN
 	1    9700 4900
@@
 F 0 "U8" H 9750 5300 60  0001 C CNN
 F 1 "Picoblade-3" H 9750 5700 60  0000 C CNN
-F 2 "Connectors_Molex:Molex_PicoBlade_53047-0310_03x1.25mm_Straight" H 9700 5350 60  0001 C CNN
+F 2 "MRDT_Connectors:MOLEX_SL_3_Vertical" H 9700 5350 60  0001 C CNN
 F 3 "" H 9700 5350 60  0001 C CNN
 	1    9700 5350
