File: DrillBoard-Hardware.kicad_pcb (KiCad board)
At the start: 2 copper layers, 23 parts, among them U1 VNH5019A-E, U2 VNH5019A-E, U3 OKI, U4 MAX-3232, U5 Molex_SL-5, U6 TM4C129E_Launchpad_X9, U7 Molex_SL-3, U8 Molex_SL-3

Commit message: Created board layout
Will run traces this wek in preparation for board review next Sunday.
Parts:
- removed 10u1, 10u2: C, Capacitors_SMD:C_0805_HandSoldering
- removed C3: .1u, Capacitors_SMD:C_0805_HandSoldering
- added C12: 10u, Capacitors_SMD:C_0603_HandSoldering, F.Cu at (128.5, 168.6)
- added C13: 1u, Capacitors_SMD:C_0603_HandSoldering, F.Cu at (138.6, 183.3)
- added C14: 1u, Capacitors_SMD:C_0603_HandSoldering, F.Cu at (137.7, 186.3)
- added C6: 47u, Capacitors_THT:CP_Radial_D5.0mm_P2.50mm, F.Cu at (160.6, 184.1)
- added C7: Anderson-2, MRDT_Connectors:Anderson_2_Horisontal_Side_by_Side, F.Cu at (118.0, 138.8)
- added C8: Anderson-2, MRDT_Connectors:Anderson_2_Horisontal_Side_by_Side, F.Cu at (162.0, 138.8)
- added G***: LOGO, MRDT_Silkscreens:Atlas_Logo_28.6mmX37.3mm, B.Cu at (146.6, 185.0)
- added G***: LOGO, MRDT_Silkscreens:MRDT_Logo_10mm, F.Cu at (136.7, 152.4)
- added REF**: Via_P1.27mm_5x5, MRDT_Drill_Holes:Via_.6m, F.Cu at (162.6, 178.8)
- added REF**: Via_P1.27mm_5x5, MRDT_Drill_Holes:Via_.6m, F.Cu at (168.9, 179.1)
- added REF**: Via_P1.27mm_5x5, MRDT_Drill_Holes:Via_.6m, F.Cu at (160.0, 156.2)
- added REF**: Via_P1.27mm_5x5, MRDT_Drill_Holes:Via_.6m, F.Cu at (158.8, 156.2)
- added REF**: Via_P1.27mm_5x5, MRDT_Drill_Holes:Via_.6m, F.Cu at (162.6, 154.9)
- added REF**: Via_P1.27mm_5x5, MRDT_Drill_Holes:Via_.6m, F.Cu at (161.3, 154.9)
- added REF**: Via_P1.27mm_5x5, MRDT_Drill_Holes:Via_.6m, F.Cu at (160.0, 154.9)
- added REF**: Via_P1.27mm_5x5, MRDT_Drill_Holes:Via_.6m, F.Cu at (158.8, 154.9)
- added REF**: Via_P1.27mm_5x5, MRDT_Drill_Holes:Via_.6m, F.Cu at (162.6, 153.7)
- added REF**: Via_P1.27mm_5x5, MRDT_Drill_Holes:Via_.6m, F.Cu at (161.3, 153.7)
- added REF**: Via_P1.27mm_5x5, MRDT_Drill_Holes:Via_.6m, F.Cu at (160.0, 153.7)
- added REF**: Via_P1.27mm_5x5, MRDT_Drill_Holes:Via_.6m, F.Cu at (158.8, 153.7)
- added REF**: Via_P1.27mm_5x5, MRDT_Drill_Holes:Via_.6m, F.Cu at (167.6, 179.1)
- added REF**: Via_P1.27mm_5x5, MRDT_Drill_Holes:Via_.6m, F.Cu at (162.6, 152.4)
- added REF**: Via_P1.27mm_5x5, MRDT_Drill_Holes:Via_.6m, F.Cu at (161.3, 152.4)
- added REF**: Via_P1.27mm_5x5, MRDT_Drill_Holes:Via_.6m, F.Cu at (160.0, 152.4)
- added REF**: Via_P1.27mm_5x5, MRDT_Drill_Holes:Via_.6m, F.Cu at (158.8, 152.4)
- added REF**: Via_P1.27mm_5x5, MRDT_Drill_Holes:Via_.6m, F.Cu at (162.6, 151.1)
- added REF**: Via_P1.27mm_5x5, MRDT_Drill_Holes:Via_.6m, F.Cu at (161.3, 151.1)
- added REF**: Via_P1.27mm_5x5, MRDT_Drill_Holes:Via_.6m, F.Cu at (160.0, 151.1)
- added REF**: Via_P1.27mm_5x5, MRDT_Drill_Holes:Via_.6m, F.Cu at (158.8, 151.1)
- added REF**: Via_P1.27mm_5x5, MRDT_Drill_Holes:Via_.6m, F.Cu at (162.6, 168.9)
- added REF**: Via_P1.27mm_5x5, MRDT_Drill_Holes:Via_.6m, F.Cu at (161.3, 168.9)
- added REF**: Via_P1.27mm_5x5, MRDT_Drill_Holes:Via_.6m, F.Cu at (166.4, 179.1)
- added REF**: Via_P1.27mm_5x5, MRDT_Drill_Holes:Via_.6m, F.Cu at (160.0, 168.9)
- added REF**: Via_P1.27mm_5x5, MRDT_Drill_Holes:Via_.6m, F.Cu at (158.8, 168.9)
- added REF**: Via_P1.27mm_5x5, MRDT_Drill_Holes:Via_.6m, F.Cu at (162.6, 170.2)
- added REF**: Via_P1.27mm_5x5, MRDT_Drill_Holes:Via_.6m, F.Cu at (161.3, 170.2)
- added REF**: Via_P1.27mm_5x5, MRDT_Drill_Holes:Via_.6m, F.Cu at (160.0, 170.2)
- added REF**: Via_P1.27mm_5x5, MRDT_Drill_Holes:Via_.6m, F.Cu at (158.8, 170.2)
- added REF**: Via_P1.27mm_5x5, MRDT_Drill_Holes:Via_.6m, F.Cu at (162.6, 171.4)
- added REF**: Via_P1.27mm_5x5, MRDT_Drill_Holes:Via_.6m, F.Cu at (161.3, 171.4)
- added REF**: Via_P1.27mm_5x5, MRDT_Drill_Holes:Via_.6m, F.Cu at (160.0, 171.4)
- added REF**: Via_P1.27mm_5x5, MRDT_Drill_Holes:Via_.6m, F.Cu at (158.8, 171.4)
- added REF**: Via_P1.27mm_5x5, MRDT_Drill_Holes:Via_.6m, F.Cu at (165.1, 179.1)
- added REF**: Via_P1.27mm_5x5, MRDT_Drill_Holes:Via_.6m, F.Cu at (162.6, 172.7)
- added REF**: Via_P1.27mm_5x5, MRDT_Drill_Holes:Via_.6m, F.Cu at (161.3, 172.7)
- added REF**: Via_P1.27mm_5x5, MRDT_Drill_Holes:Via_.6m, F.Cu at (160.0, 172.7)
- added REF**: Via_P1.27mm_5x5, MRDT_Drill_Holes:Via_.6m, F.Cu at (158.8, 172.7)
- added REF**: Via_P1.27mm_5x5, MRDT_Drill_Holes:Via_.6m, F.Cu at (162.6, 174.0)
- added REF**: Via_P1.27mm_5x5, MRDT_Drill_Holes:Via_.6m, F.Cu at (161.3, 174.0)
- added REF**: Via_P1.27mm_5x5, MRDT_Drill_Holes:Via_.6m, F.Cu at (160.0, 174.0)
- added REF**: Via_P1.27mm_5x5, MRDT_Drill_Holes:Via_.6m, F.Cu at (158.8, 174.0)
- added REF**: Via_P1.27mm_5x5, MRDT_Drill_Holes:Via_.6m, F.Cu at (162.6, 175.3)
- added REF**: Via_P1.27mm_5x5, MRDT_Drill_Holes:Via_.6m, F.Cu at (161.3, 175.3)
- added REF**: Via_P1.27mm_5x5, MRDT_Drill_Holes:Via_.6m, F.Cu at (168.9, 177.8)
- added REF**: Via_P1.27mm_5x5, MRDT_Drill_Holes:Via_.6m, F.Cu at (160.0, 175.3)
- added REF**: Via_P1.27mm_5x5, MRDT_Drill_Holes:Via_.6m, F.Cu at (158.8, 175.3)
- added REF**: Via_P1.27mm_5x5, MRDT_Drill_Holes:Via_.6m, F.Cu at (162.6, 176.5)
- added REF**: Via_P1.27mm_5x5, MRDT_Drill_Holes:Via_.6m, F.Cu at (161.3, 176.5)
- added REF**: Via_P1.27mm_5x5, MRDT_Drill_Holes:Via_.6m, F.Cu at (160.0, 176.5)
- added REF** (x2): Via_P1.27mm_5x5, MRDT_Drill_Holes:Via_.6m, F.Cu at (158.8, 176.5)
- added REF**: Via_P1.27mm_5x5, MRDT_Drill_Holes:Via_.6m, F.Cu at (162.6, 177.8)
- added REF**: Via_P1.27mm_5x5, MRDT_Drill_Holes:Via_.6m, F.Cu at (161.3, 177.8)
- added REF**: Via_P1.27mm_5x5, MRDT_Drill_Holes:Via_.6m, F.Cu at (160.0, 177.8)
- added REF**: Via_P1.27mm_5x5, MRDT_Drill_Holes:Via_.6m, F.Cu at (158.8, 177.8)
- added REF**: Via_P1.27mm_5x5, MRDT_Drill_Holes:Via_.6m, F.Cu at (167.6, 177.8)
- added REF**: Via_P1.27mm_5x5, MRDT_Drill_Holes:Via_.6m, F.Cu at (166.4, 177.8)
- added REF**: Via_P1.27mm_5x5, MRDT_Drill_Holes:Via_.6m, F.Cu at (165.1, 177.8)
- added REF**: Via_P1.27mm_5x5, MRDT_Drill_Holes:Via_.6m, F.Cu at (168.9, 176.5)
- added REF**: Via_P1.27mm_5x5, MRDT_Drill_Holes:Via_.6m, F.Cu at (167.6, 176.5)
- added REF**: Via_P1.27mm_5x5, MRDT_Drill_Holes:Via_.6m, F.Cu at (161.3, 178.8)
- added REF**: Via_P1.27mm_5x5, MRDT_Drill_Holes:Via_.6m, F.Cu at (166.4, 176.5)
- added REF**: Via_P1.27mm_5x5, MRDT_Drill_Holes:Via_.6m, F.Cu at (165.1, 176.5)
- added REF**: Via_P1.27mm_5x5, MRDT_Drill_Holes:Via_.6m, F.Cu at (168.9, 175.3)
- added REF**: Via_P1.27mm_5x5, MRDT_Drill_Holes:Via_.6m, F.Cu at (167.6, 175.3)
- added REF**: Via_P1.27mm_5x5, MRDT_Drill_Holes:Via_.6m, F.Cu at (166.4, 175.3)
- added REF**: Via_P1.27mm_5x5, MRDT_Drill_Holes:Via_.6m, F.Cu at (165.1, 175.3)
- added REF**: Via_P1.27mm_5x5, MRDT_Drill_Holes:Via_.6m, F.Cu at (168.9, 172.7)
- added REF**: Via_P1.27mm_5x5, MRDT_Drill_Holes:Via_.6m, F.Cu at (167.6, 172.7)
- added REF**: Via_P1.27mm_5x5, MRDT_Drill_Holes:Via_.6m, F.Cu at (166.4, 172.7)
- added REF**: Via_P1.27mm_5x5, MRDT_Drill_Holes:Via_.6m, F.Cu at (165.1, 172.7)
- added REF**: Via_P1.27mm_5x5, MRDT_Drill_Holes:Via_.6m, F.Cu at (160.0, 178.8)
- added REF**: Via_P1.27mm_5x5, MRDT_Drill_Holes:Via_.6m, F.Cu at (168.9, 171.4)
- added REF**: Via_P1.27mm_5x5, MRDT_Drill_Holes:Via_.6m, F.Cu at (167.6, 171.4)
- added REF**: Via_P1.27mm_5x5, MRDT_Drill_Holes:Via_.6m, F.Cu at (166.4, 171.4)
- added REF**: Via_P1.27mm_5x5, MRDT_Drill_Holes:Via_.6m, F.Cu at (165.1, 171.4)
- added REF**: Via_P1.27mm_5x5, MRDT_Drill_Holes:Via_.6m, F.Cu at (168.9, 170.2)
- added REF**: Via_P1.27mm_5x5, MRDT_Drill_Holes:Via_.6m, F.Cu at (167.6, 170.2)
- added REF**: Via_P1.27mm_5x5, MRDT_Drill_Holes:Via_.6m, F.Cu at (166.4, 170.2)
- added REF**: Via_P1.27mm_5x5, MRDT_Drill_Holes:Via_.6m, F.Cu at (165.1, 170.2)
- added REF**: Via_P1.27mm_5x5, MRDT_Drill_Holes:Via_.6m, F.Cu at (168.9, 168.9)
- added REF**: Via_P1.27mm_5x5, MRDT_Drill_Holes:Via_.6m, F.Cu at (167.6, 168.9)
- added REF**: Via_P1.27mm_5x5, MRDT_Drill_Holes:Via_.6m, F.Cu at (158.8, 178.8)
- added REF**: Via_P1.27mm_5x5, MRDT_Drill_Holes:Via_.6m, F.Cu at (166.4, 168.9)
- added REF**: Via_P1.27mm_5x5, MRDT_Drill_Holes:Via_.6m, F.Cu at (165.1, 168.9)
- added REF**: Via_P1.27mm_5x5, MRDT_Drill_Holes:Via_.6m, F.Cu at (168.9, 167.6)
- added REF**: Via_P1.27mm_5x5, MRDT_Drill_Holes:Via_.6m, F.Cu at (167.6, 167.6)
- added REF**: Via_P1.27mm_5x5, MRDT_Drill_Holes:Via_.6m, F.Cu at (166.4, 167.6)
- added REF**: Via_P1.27mm_5x5, MRDT_Drill_Holes:Via_.6m, F.Cu at (165.1, 167.6)
- added REF**: Via_P1.27mm_5x5, MRDT_Drill_Holes:Via_.6m, F.Cu at (156.2, 162.6)
- added REF**: Via_P1.27mm_5x5, MRDT_Drill_Holes:Via_.6m, F.Cu at (154.9, 162.6)
- added REF**: Via_P1.27mm_5x5, MRDT_Drill_Holes:Via_.6m, F.Cu at (153.7, 162.6)
- added REF**: Via_P1.27mm_5x5, MRDT_Drill_Holes:Via_.6m, F.Cu at (152.4, 162.6)
- added REF**: Via_P1.27mm_5x5, MRDT_Drill_Holes:Via_.6m, F.Cu at (156.2, 161.3)
- added REF**: Via_P1.27mm_5x5, MRDT_Drill_Holes:Via_.6m, F.Cu at (154.9, 161.3)
- added REF**: Via_P1.27mm_5x5, MRDT_Drill_Holes:Via_.6m, F.Cu at (153.7, 161.3)
- added REF**: Via_P1.27mm_5x5, MRDT_Drill_Holes:Via_.6m, F.Cu at (152.4, 161.3)
- added REF**: Via_P1.27mm_5x5, MRDT_Drill_Holes:Via_.6m, F.Cu at (156.2, 160.0)
- added REF**: Via_P1.27mm_5x5, MRDT_Drill_Holes:Via_.6m, F.Cu at (154.9, 160.0)
- added REF**: Via_P1.27mm_5x5, MRDT_Drill_Holes:Via_.6m, F.Cu at (153.7, 160.0)
- added REF**: Via_P1.27mm_5x5, MRDT_Drill_Holes:Via_.6m, F.Cu at (152.4, 160.0)
- added REF**: Via_P1.27mm_5x5, MRDT_Drill_Holes:Via_.6m, F.Cu at (156.2, 158.8)
- added REF**: Via_P1.27mm_5x5, MRDT_Drill_Holes:Via_.6m, F.Cu at (154.9, 158.8)
- added REF**: Via_P1.27mm_5x5, MRDT_Drill_Holes:Via_.6m, F.Cu at (168.9, 180.3)
- added REF**: Via_P1.27mm_5x5, MRDT_Drill_Holes:Via_.6m, F.Cu at (153.7, 158.8)
- added REF**: Via_P1.27mm_5x5, MRDT_Drill_Holes:Via_.6m, F.Cu at (152.4, 158.8)
- added REF**: Via_P1.27mm_5x5, MRDT_Drill_Holes:Via_.6m, F.Cu at (156.2, 157.5)
- added REF**: Via_P1.27mm_5x5, MRDT_Drill_Holes:Via_.6m, F.Cu at (154.9, 157.5)
- added REF**: Via_P1.27mm_5x5, MRDT_Drill_Holes:Via_.6m, F.Cu at (153.7, 157.5)
- added REF**: Via_P1.27mm_5x5, MRDT_Drill_Holes:Via_.6m, F.Cu at (152.4, 157.5)
- added REF**: Via_P1.27mm_5x5, MRDT_Drill_Holes:Via_.6m, F.Cu at (156.2, 153.7)
- added REF**: Via_P1.27mm_5x5, MRDT_Drill_Holes:Via_.6m, F.Cu at (154.9, 153.7)
- added REF**: Via_P1.27mm_5x5, MRDT_Drill_Holes:Via_.6m, F.Cu at (153.7, 153.7)
- added REF**: Via_P1.27mm_5x5, MRDT_Drill_Holes:Via_.6m, F.Cu at (152.4, 153.7)
- added REF**: Via_P1.27mm_5x5, MRDT_Drill_Holes:Via_.6m, F.Cu at (167.6, 180.3)
- added REF**: Via_P1.27mm_5x5, MRDT_Drill_Holes:Via_.6m, F.Cu at (156.2, 152.4)
- added REF**: Via_P1.27mm_5x5, MRDT_Drill_Holes:Via_.6m, F.Cu at (154.9, 152.4)
- added REF**: Via_P1.27mm_5x5, MRDT_Drill_Holes:Via_.6m, F.Cu at (153.7, 152.4)
- added REF**: Via_P1.27mm_5x5, MRDT_Drill_Holes:Via_.6m, F.Cu at (152.4, 152.4)
- added REF**: Via_P1.27mm_5x5, MRDT_Drill_Holes:Via_.6m, F.Cu at (156.2, 151.1)
- added REF**: Via_P1.27mm_5x5, MRDT_Drill_Holes:Via_.6m, F.Cu at (154.9, 151.1)
- added REF**: Via_P1.27mm_5x5, MRDT_Drill_Holes:Via_.6m, F.Cu at (153.7, 151.1)
- added REF**: Via_P1.27mm_5x5, MRDT_Drill_Holes:Via_.6m, F.Cu at (152.4, 151.1)
- added REF**: Via_P1.27mm_5x5, MRDT_Drill_Holes:Via_.6m, F.Cu at (156.2, 149.9)
- added REF**: Via_P1.27mm_5x5, MRDT_Drill_Holes:Via_.6m, F.Cu at (154.9, 149.9)
- added REF**: Via_P1.27mm_5x5, MRDT_Drill_Holes:Via_.6m, F.Cu at (166.4, 180.3)
- added REF**: Via_P1.27mm_5x5, MRDT_Drill_Holes:Via_.6m, F.Cu at (153.7, 149.9)
- added REF**: Via_P1.27mm_5x5, MRDT_Drill_Holes:Via_.6m, F.Cu at (152.4, 149.9)
- added REF**: Via_P1.27mm_5x5, MRDT_Drill_Holes:Via_.6m, F.Cu at (156.2, 148.6)
- added REF**: Via_P1.27mm_5x5, MRDT_Drill_Holes:Via_.6m, F.Cu at (154.9, 148.6)
- added REF**: Via_P1.27mm_5x5, MRDT_Drill_Holes:Via_.6m, F.Cu at (153.7, 148.6)
- added REF**: Via_P1.27mm_5x5, MRDT_Drill_Holes:Via_.6m, F.Cu at (152.4, 148.6)
- added REF**: Via_P1.27mm_5x5, MRDT_Drill_Holes:Via_.6m, F.Cu at (162.6, 160.0)
- added REF**: Via_P1.27mm_5x5, MRDT_Drill_Holes:Via_.6m, F.Cu at (161.3, 160.0)
- added REF**: Via_P1.27mm_5x5, MRDT_Drill_Holes:Via_.6m, F.Cu at (160.0, 160.0)
- added REF**: Via_P1.27mm_5x5, MRDT_Drill_Holes:Via_.6m, F.Cu at (158.8, 160.0)
- added REF**: Via_P1.27mm_5x5, MRDT_Drill_Holes:Via_.6m, F.Cu at (165.1, 180.3)
- added REF**: Via_P1.27mm_5x5, MRDT_Drill_Holes:Via_.6m, F.Cu at (162.6, 158.8)
- added REF**: Via_P1.27mm_5x5, MRDT_Drill_Holes:Via_.6m, F.Cu at (161.3, 158.8)
- added REF**: Via_P1.27mm_5x5, MRDT_Drill_Holes:Via_.6m, F.Cu at (160.0, 158.8)
- added REF**: Via_P1.27mm_5x5, MRDT_Drill_Holes:Via_.6m, F.Cu at (158.8, 158.8)
- added REF**: Via_P1.27mm_5x5, MRDT_Drill_Holes:Via_.6m, F.Cu at (162.6, 157.5)
- added REF**: Via_P1.27mm_5x5, MRDT_Drill_Holes:Via_.6m, F.Cu at (161.3, 157.5)
- added REF**: Via_P1.27mm_5x5, MRDT_Drill_Holes:Via_.6m, F.Cu at (160.0, 157.5)
- added REF**: Via_P1.27mm_5x5, MRDT_Drill_Holes:Via_.6m, F.Cu at (158.8, 157.5)
- added REF**: Via_P1.27mm_5x5, MRDT_Drill_Holes:Via_.6m, F.Cu at (162.6, 156.2)
- added REF**: Via_P1.27mm_5x5, MRDT_Drill_Holes:Via_.6m, F.Cu at (161.3, 156.2)
- added SW1: 3P1T_Fused, MRDT_Switches:3P1T_Switch, F.Cu at (154.6, 204.9)
- C1: footprint MRDT-Connectors:Anderson_3_Horisontal_Side-by-Side -> MRDT_Connectors:Anderson_3_Horisontal_Side_by_Side
- C10, C11, C4, C9: footprint Capacitors_SMD:C_0805_HandSoldering -> Capacitors_SMD:C_0603_HandSoldering
- C2: value Anderson-3 -> 10u; footprint MRDT-Connectors:Anderson_3_Horisontal_Side-by-Side -> Capacitors_SMD:C_0603_HandSoldering
- R1, R2, R3, R4, R5, R6: footprint Resistors_SMD:R_0805_HandSoldering -> Resistors_SMD:R_0603_HandSoldering
- U1, U2: footprint MRDT-ICs:MultiPowerSO-30 -> MRDT_ICs:MultiPowerSO_30
- U3: footprint MRDT-Devices:OKI -> MRDT_Devices:OKI_Horisontal
- U5: footprint MRDT-Connectors:MOLEX_SL_5 -> MRDT_Connectors:MOLEX_SL_5
- U6: footprint MRDT-Shields:TM4C129E_Launchpad_X9 -> MRDT_Shields:TM4C129E_Launchpad_X9
- U7, U8: value Molex_SL-3 -> Picoblade-3; footprint MRDT-connectors:MOLEX_SL_3 -> Connectors_Molex:Molex_PicoBlade_53047-0310_03x1.25mm_Straight
- moved C2 142.5 mm to (128.5, 174.0), turned to 90 degrees
- moved C10 137.9 mm to (139.6, 186.2), turned to 270 degrees
- moved C9 135.7 mm to (135.1, 183.3), turned to 270 degrees
- moved U3 135.3 mm to (131.4, 176.7), turned to 90 degrees
- moved U5 134.6 mm to (131.3, 193.0), turned to 90 degrees
- moved U4 127.9 mm to (144.3, 186.4), turned to 0 degrees
- moved U7 124.7 mm to (120.2, 172.7), turned to 0 degrees
- moved U8 123.3 mm to (120.3, 181.5), turned to 0 degrees
- moved U6 109.1 mm to (118.0, 208.6)
- moved C4 107.3 mm to (165.4, 184.2)
- moved R6 102.4 mm to (150.4, 175.8)
- moved R5 97.4 mm to (150.4, 172.8)
- moved R4 91.9 mm to (150.4, 169.9)
- moved C1 82.2 mm to (136.3, 138.8)
- moved C11 81.9 mm to (146.2, 180.1)
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Connections:
- net Net-(C7-Pad1) renamed /Out_A1
- net Net-(C7-Pad2) renamed /Out_B1
- net Net-(C8-Pad1) renamed /Out_A2
- net Net-(C8-Pad2) renamed /Out_B2
- C1 pad 2: Net-(10u1-Pad1) -> /12V_Logic
- C11 pad 2: Net-(C11-Pad2) -> (no net)
- C2 pad 1: Net-(C2-Pad1) -> /12V_Logic
- C2 pad 2: Net-(C2-Pad2) -> GND
- U1 pad 11: Net-(U1-Pad11) -> (no net)
- U1 pad 14: Net-(U1-Pad14) -> (no net)
- U1 pad 17: Net-(U1-Pad17) -> (no net)
- U1 pad 2: Net-(U1-Pad2) -> (no net)
- U1 pad 22: Net-(U1-Pad22) -> (no net)
- U1 pad 24: Net-(U1-Pad24) -> (no net)
- U1 pad 29: Net-(U1-Pad29) -> (no net)
- U1 pad 8: Net-(U1-Pad8) -> (no net)
- U2 pad 11: Net-(U2-Pad11) -> (no net)
- U2 pad 14: Net-(U2-Pad14) -> (no net)
- U2 pad 17: Net-(U2-Pad17) -> (no net)
- U2 pad 2: Net-(U2-Pad2) -> (no net)
- U2 pad 22: Net-(U2-Pad22) -> (no net)
- U2 pad 24: Net-(U2-Pad24) -> (no net)
- U2 pad 29: Net-(U2-Pad29) -> (no net)
- U2 pad 8: Net-(U2-Pad8) -> (no net)
- U3 pad 1: Net-(10u1-Pad1) -> /12V_Logic
- U4 pad 11: Net-(U4-Pad11) -> (no net)
- U4 pad 12: Net-(U4-Pad12) -> (no net)
- U4 pad 13: Net-(U4-Pad13) -> (no net)
- U4 pad 14: Net-(U4-Pad14) -> (no net)
- U5 pad 4: Net-(U5-Pad4) -> (no net)
- U5 pad 5: Net-(U5-Pad5) -> (no net)
- U6 pad PA6: Net-(U6-PadPA6) -> (no net)
- U6 pad PB2: Net-(U6-PadPB2) -> (no net)
- U6 pad PB3: Net-(U6-PadPB3) -> (no net)
- U6 pad PC6: Net-(U6-PadPC6) -> (no net)
- U6 pad PD3: Net-(U6-PadPD3) -> (no net)
- U6 pad PD7: Net-(U6-PadPD7) -> (no net)
- U6 pad PE0: Net-(U6-PadPE0) -> (no net)
- U6 pad PE1: Net-(U6-PadPE1) -> (no net)
- U6 pad PE2: Net-(U6-PadPE2) -> (no net)
- U6 pad PE3: Net-(U6-PadPE3) -> (no net)
- U6 pad PE4: Net-(U6-PadPE4) -> (no net)
- U6 pad PE5: Net-(U6-PadPE5) -> (no net)
- U6 pad PF1: Net-(U6-PadPF1) -> (no net)
- U6 pad PF2: Net-(U6-PadPF2) -> (no net)
- U6 pad PF3: Net-(U6-PadPF3) -> (no net)
- U6 pad PG0: Net-(U6-PadPG0) -> (no net)
- U6 pad PL2: Net-(U6-PadPL2) -> (no net)
- U6 pad PL3: Net-(U6-PadPL3) -> (no net)
- U6 pad PL4: Net-(U6-PadPL4) -> (no net)
- U6 pad PM3: Net-(U6-PadPM3) -> (no net)
- U6 pad PM4: Net-(U6-PadPM4) -> (no net)
- U6 pad PN2: Net-(U6-PadPN2) -> (no net)
- U6 pad PN3: Net-(U6-PadPN3) -> (no net)
- U6 pad PP2: Net-(U6-PadPP2) -> (no net)
- U6 pad Rese: Net-(U6-PadRese) -> (no net)
- U7 pad 1: GND -> +3V3
- U7 pad 3: +3V3 -> GND
- U8 pad 1: GND -> +3V3
- U8 pad 3: +3V3 -> GND
Routing:
- net +3V3: track 87.8 -> 0.00 mm
- net PWM1: track 52.4 -> 0.00 mm
- net Encoder1_PWM: track 38.1 -> 0.00 mm
- net Encoder2_PWM: track 31.6 -> 0.00 mm
- net Net-(U4-Pad7): track 30.2 -> 0.00 mm
- net IN_A1: track 27.5 -> 0.00 mm, vias 1 -> 0
- net Net-(U4-Pad8): track 26.7 -> 0.00 mm
- net IN_B1: track 25.6 -> 0.00 mm
- net +12V: track 0.00 -> 23.8 mm
- net /Out_A2: track 0.00 -> 6.85 mm
- net Net-(C10-Pad2): track 6.38 -> 0.00 mm
- net Net-(R2-Pad1): track 6.09 -> 0.00 mm
- net Net-(R3-Pad1): track 5.50 -> 0.00 mm
- net /Out_B2: track 0.00 -> 5.43 mm
- net /Out_B1: track 0.00 -> 5.41 mm
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- added copper zone on B.Cu, net +12V
- added copper zone on F.Cu, net +12V
- added copper zone on B.Cu, net /Out_A1
- added copper zone on F.Cu, net /Out_A1
- added copper zone on B.Cu, net /Out_A2
- added copper zone on F.Cu, net /Out_A2
- added copper zone on B.Cu, net /Out_B1
- added copper zone on F.Cu, net /Out_B1
- added copper zone on B.Cu, net /Out_B2
- added copper zone on F.Cu, net /Out_B2
- added copper zone on F.Cu, net GND
Other:
- board outline added: 59.7 x 109.8 mm
- board text added: "Brushed DC Motor Driver, Rev 1 Mars Rover Design Team, 2018 Missouri S&T Andrew Van Horn, Jacob Lipina"
- board text added: "Drives: 2 independant motors @ 13A 1 motor in Parallel @ 26A"
- board text added: "ENC 1"
- board text added: "ENC 2"
- board text added: "Independant"
- board text added: "Parallel"

Commit message: Finished Board
Parts:
- added G***: LOGO, MRDT_Silkscreens:Andrew_Van_Horn_Sig_15mm, B.Cu at (128.5, 214.8)
- moved C11 0.14 mm to (146.1, 180.1)
- moved U7 0.11 mm to (120.3, 172.7)
- turned R5 to 180 degrees
- turned R4 to 180 degrees
- turned R6 to 180 degrees
Routing:
- net IN_B1: track 0.00 -> 151.2 mm, vias 0 -> 4
- net +3V3: track 0.00 -> 147.9 mm, vias 0 -> 4
- net IN_A1: track 0.00 -> 130.0 mm, vias 0 -> 2
- net PWM1: track 0.00 -> 84.7 mm, vias 0 -> 2
- net IN_B2: track 0.00 -> 58.9 mm, vias 0 -> 1
- net PWM2: track 0.00 -> 50.1 mm, vias 0 -> 2
- net /12V_Logic: track 0.00 -> 49.2 mm, vias 0 -> 2
- net IN_A2: track 0.00 -> 45.9 mm, vias 0 -> 2
- net TX: track 0.00 -> 33.5 mm
- net RX: track 0.00 -> 30.8 mm
- net Encoder2_PWM: track 0.00 -> 30.4 mm, vias 0 -> 1
- net Encoder1_PWM: track 0.00 -> 19.6 mm, vias 0 -> 1
- net Net-(U4-Pad8): track 0.00 -> 13.3 mm
- net Net-(U4-Pad7): track 0.00 -> 12.8 mm
- net GND: track 0.00 -> 10.3 mm, vias 0 -> 2
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- added copper zone on F.Cu, net +3V3
- added copper zone on B.Cu, net GND
Other:
- board text added: "Motor 1"
- board text added: "Motor 2"
- board text added: "Serial"

Commit message: Finalized schematic and board and generated Gerbs
Parts:
- removed C10, C11, C13, C14: 1u, Capacitors_SMD:C_0603_HandSoldering
- added C3: 10u, Capacitors_SMD:C_0603_HandSoldering, F.Cu at (163.4, 185.0)
- added C5: 10u, Capacitors_SMD:C_0603_HandSoldering, F.Cu at (159.7, 185.0)
- added G***: LOGO, MRDT_Silkscreens:Jacob_Lipina_Sig_15mm, F.Cu at (148.9, 223.9)
- added R10: 10K, Resistors_SMD:R_0603_HandSoldering, F.Cu at (128.0, 198.1)
- added R7: 10K, Resistors_SMD:R_0603_HandSoldering, F.Cu at (133.3, 198.1)
- added R8: 10K, Resistors_SMD:R_0603_HandSoldering, F.Cu at (131.6, 198.1)
- added R9: 10K, Resistors_SMD:R_0603_HandSoldering, F.Cu at (129.8, 198.1)
- added REF**: Via_P1.27mm_5x5, MRDT_Drill_Holes:Via_.6m, F.Cu at (144.6, 163.0)
- added REF**: Via_P1.27mm_5x5, MRDT_Drill_Holes:Via_.6m, F.Cu at (145.8, 161.8)
- added REF**: Via_P1.27mm_5x5, MRDT_Drill_Holes:Via_.6m, F.Cu at (144.6, 161.8)
- added REF**: Via_P1.27mm_5x5, MRDT_Drill_Holes:Via_.6m, F.Cu at (145.8, 163.0)
- added U10: LS_4, MRDT_Connectors:MOLEX_SL_2_Vertical, F.Cu at (122.2, 196.6)
- added U9: LS_3, MRDT_Connectors:MOLEX_SL_2_Vertical, F.Cu at (122.2, 188.8)
- C1: value Anderson-3 -> Anderson_3
- C6: value 47u -> 10u; footprint Capacitors_THT:CP_Radial_D5.0mm_P2.50mm -> Capacitors_SMD:C_0603_HandSoldering
- C9: value 1u -> 10u
- G***: moved to F.Cu
- U4: value MAX-3232 -> LS_1; footprint Housings_SOIC:SOIC-16_3.9x9.9mm_Pitch1.27mm -> MRDT_Connectors:MOLEX_SL_2_Vertical
- U5: value Molex_SL-5 -> LS_2; footprint MRDT_Connectors:MOLEX_SL_5 -> MRDT_Connectors:MOLEX_SL_2_Vertical
- U7, U8: footprint Connectors_Molex:Molex_PicoBlade_53047-0310_03x1.25mm_Straight -> MRDT_Connectors:MOLEX_SL_3_Vertical
- moved SW1 43.1 mm to (135.0, 166.5), turned to 270 degrees
- moved U8 30.2 mm to (147.3, 194.9)
- moved C9 29.7 mm to (164.8, 185.0)
- moved U7 27.2 mm to (135.9, 194.9)
- moved U4 25.7 mm to (122.2, 173.4), turned to 90 degrees
- moved U5 15.0 mm to (122.2, 181.1)
- moved C12 13.9 mm to (134.4, 181.2)
- moved C2 12.8 mm to (134.4, 185.4)
- moved U3 12.6 mm to (136.3, 188.3)
- moved G*** 9.05 mm to (130.4, 223.7), turned to 0 degrees
- moved C4 3.49 mm to (162.0, 185.0), turned to 270 degrees
- moved C6 2.51 mm to (158.2, 185.0)
Connections:
- C9 pad 1: Net-(C9-Pad1) -> +12V
- C9 pad 2: Net-(C9-Pad2) -> GND
- U4 pad 1: Net-(C9-Pad1) -> +3V3
- U4 pad 2: Net-(C13-Pad2) -> LS_1
- U5 pad 1: Net-(U4-Pad8) -> +3V3
- U5 pad 2: Net-(U4-Pad7) -> LS_2
- U6 pad PC4: RX -> (no net)
- U6 pad PC5: TX -> (no net)
- U6 pad PD0: Encoder2_PWM -> Encoder1_PWM
- U6 pad PD1: Encoder1_PWM -> Encoder2_PWM
- U6 pad PE0: (no net) -> LS_4
- U6 pad PE1: (no net) -> LS_3
- U6 pad PE2: (no net) -> LS_2
- U6 pad PE3: (no net) -> LS_1
- U6 pad PF1: (no net) -> PWM1
- U6 pad PF2: (no net) -> PWM2
- U6 pad PL5: PWM2 -> (no net)
- U6 pad PM5: PWM1 -> (no net)
Routing:
- net IN_A1: track 130.0 -> 48.3 mm, vias 2 -> 0
- net IN_B1: track 151.2 -> 71.0 mm, vias 4 -> 0
- net LS_1: track 0.00 -> 39.4 mm
- net +3V3: track 147.9 -> 183.4 mm
- net LS_2: track 0.00 -> 34.3 mm
- net TX: track 33.5 -> 0.00 mm
- net RX: track 30.8 -> 0.00 mm
- net Encoder2_PWM: track 30.4 -> 58.7 mm, vias 1 -> 0
- net Encoder1_PWM: track 19.6 -> 45.5 mm, vias 1 -> 0
- net LS_3: track 0.00 -> 25.4 mm
- net IN_A2: track 45.9 -> 21.8 mm, vias 2 -> 1
- net IN_B2: track 58.9 -> 35.1 mm
- net /12V_Logic: track 49.2 -> 70.3 mm, vias 2 -> 3
- net +12V: track 23.8 -> 41.0 mm, vias 0 -> 1
- net LS_4: track 0.00 -> 16.4 mm
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- removed copper zone on F.Cu, net +3V3
Other:
- board text added: "Ind."
- board text added: "LS-1"
- board text added: "LS-2"
- board text added: "LS-3"
- board text added: "LS-4"
- board text removed: "Independant"
- board text removed: "Serial"

Commit message: Added Power LED and Gerbs
Parts:
- added D1: LED, Diodes_SMD:D_1206, F.Cu at (130.2, 176.1)
- added R11: 330, Resistors_SMD:R_0603_HandSoldering, F.Cu at (135.8, 177.5)
Routing:
- net Net-(D1-Pad2): track 0.00 -> 3.65 mm
- net +3V3: track 183.4 -> 186.8 mm
- net GND: track 0.00 -> 2.92 mm, vias 0 -> 1
Other:
- board text added: "Power"
Changed lines of the file:
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@@
 (kicad_pcb (version 4) (host pcbnew 4.0.7)
   (general
-    (links 0)
+    (links 259)
     (no_connects 0)
-    (area 116.32154 81.433999 179.73926 234.209661)
+    (area 117.958399 124.130599 177.748401 234.034801)
     (thickness 1.6)
-    (drawings 30)
-    (tracks 253)
+    (drawings 31)
+    (tracks 261)
     (zones 0)
-    (modules 188)
-    (nets 27)
+    (modules 190)
+    (nets 28)
   )
   (page A4 portrait)
@@
   (net 25 LS_3)
   (net 26 LS_4)
+  (net 27 "Net-(D1-Pad2)")
   (net_class Default "This is the default net class."
     (clearance 0.14986)
@@
     (add_net LS_3)
     (add_net LS_4)
+    (add_net "Net-(D1-Pad2)")
     (add_net "Net-(R1-Pad1)")
     (add_net "Net-(R2-Pad1)")
@@
       (xy -5.922912 2.000037)) (layer F.SilkS) (width 0.01))
   )
+  (module Diodes_SMD:D_1206 (layer F.Cu)
+    (at 130.175 176.149)
+    (descr "Diode SMD 1206, reflow soldering http://datasheets.avx.com/schottky.pdf")
+    (tags "Diode 1206")
+    (attr smd)
+    (fp_text reference D1 (at 0 -1.8) (layer F.SilkS)
+      (effects (font (size 1 1) (thickness 0.15)))
+    )
+    (fp_text value LED (at 0 1.9) (layer F.Fab)
+      (effects (font (size 1 1) (thickness 0.15)))
+    )
+    (fp_text user %R (at 0 -1.8) (layer F.Fab)
+      (effects (font (size 1 1) (thickness 0.15)))
+    )
+    (fp_line (start -0.254 -0.254) (end -0.254 0.254) (layer F.Fab) (width 0.1))
+    (fp_line (start 0.127 0) (end 0.381 0) (layer F.Fab) (width 0.1))
+    (fp_line (start -0.254 0) (end -0.508 0) (layer F.Fab) (width 0.1))
+    (fp_line (start 0.127 0.254) (end -0.254 0) (layer F.Fab) (width 0.1))
+    (fp_line (start 0.127 -0.254) (end 0.127 0.254) (layer F.Fab) (width 0.1))
+    (fp_line (start -0.254 0) (end 0.127 -0.254) (layer F.Fab) (width 0.1))
+    (fp_line (start -2.2 -1.06) (end -2.2 1.06) (layer F.SilkS) (width 0.12))
+    (fp_line (start -1.7 0.95) (end -1.7 -0.95) (layer F.Fab) (width 0.1))
+    (fp_line (start 1.7 0.95) (end -1.7 0.95) (layer F.Fab) (width 0.1))
+    (fp_line (start 1.7 -0.95) (end 1.7 0.95) (layer F.Fab) (width 0.1))
+    (fp_line (start -1.7 -0.95) (end 1.7 -0.95) (layer F.Fab) (width 0.1))
+    (fp_line (start -2.3 -1.16) (end 2.3 -1.16) (layer F.CrtYd) (width 0.05))
+    (fp_line (start -2.3 1.16) (end 2.3 1.16) (layer F.CrtYd) (width 0.05))
+    (fp_line (start -2.3 -1.16) (end -2.3 1.16) (layer F.CrtYd) (width 0.05))
+    (fp_line (start 2.3 -1.16) (end 2.3 1.16) (layer F.CrtYd) (width 0.05))
+    (fp_line (start 1 -1.06) (end -2.2 -1.06) (layer F.SilkS) (width 0.12))
+    (fp_line (start -2.2 1.06) (end 1 1.06) (layer F.SilkS) (width 0.12))
+    (pad 1 smd rect (at -1.5 0) (size 1 1.6) (layers F.Cu F.Paste F.Mask)
+      (net 1 GND))
+    (pad 2 smd rect (at 1.5 0) (size 1 1.6) (layers F.Cu F.Paste F.Mask)
+      (net 27 "Net-(D1-Pad2)"))
+    (model ${KISYS3DMOD}/Diodes_SMD.3dshapes/D_1206.wrl
+      (at (xyz 0 0 0))
+      (scale (xyz 1 1 1))
+      (rotate (xyz 0 0 0))
+    )
+  )
+  (module Resistors_SMD:R_0603_HandSoldering (layer F.Cu)
+    (at 135.847 177.546)
+    (descr "Resistor SMD 0603, hand soldering")
+    (tags "resistor 0603")
+    (attr smd)
+    (fp_text reference R11 (at 0 -1.45) (layer F.SilkS)
+      (effects (font (size 1 1) (thickness 0.15)))
+    )
+    (fp_text value 330 (at 0 1.55) (layer F.Fab)
+      (effects (font (size 1 1) (thickness 0.15)))
+    )
+    (fp_text user %R (at 0 0) (layer F.Fab)
+      (effects (font (size 0.4 0.4) (thickness 0.075)))
+    )
+    (fp_line (start -0.8 0.4) (end -0.8 -0.4) (layer F.Fab) (width 0.1))
+    (fp_line (start 0.8 0.4) (end -0.8 0.4) (layer F.Fab) (width 0.1))
+    (fp_line (start 0.8 -0.4) (end 0.8 0.4) (layer F.Fab) (width 0.1))
+    (fp_line (start -0.8 -0.4) (end 0.8 -0.4) (layer F.Fab) (width 0.1))
+    (fp_line (start 0.5 0.68) (end -0.5 0.68) (layer F.SilkS) (width 0.12))
+    (fp_line (start -0.5 -0.68) (end 0.5 -0.68) (layer F.SilkS) (width 0.12))
+    (fp_line (start -1.96 -0.7) (end 1.95 -0.7) (layer F.CrtYd) (width 0.05))
+    (fp_line (start -1.96 -0.7) (end -1.96 0.7) (layer F.CrtYd) (width 0.05))
+    (fp_line (start 1.95 0.7) (end 1.95 -0.7) (layer F.CrtYd) (width 0.05))
+    (fp_line (start 1.95 0.7) (end -1.96 0.7) (layer F.CrtYd) (width 0.05))
+    (pad 1 smd rect (at -1.1 0) (size 1.2 0.9) (layers F.Cu F.Paste F.Mask)
+      (net 27 "Net-(D1-Pad2)"))
+    (pad 2 smd rect (at 1.1 0) (size 1.2 0.9) (layers F.Cu F.Paste F.Mask)
+      (net 2 +3V3))
+    (model ${KISYS3DMOD}/Resistors_SMD.3dshapes/R_0603.wrl
+      (at (xyz 0 0 0))
+      (scale (xyz 1 1 1))
+      (rotate (xyz 0 0 0))
+    )
+  )
+  (gr_text Power (at 130.556 178.435) (layer F.SilkS)
+    (effects (font (size 1.5 1.5) (thickness 0.3)))
+  )
   (gr_text LS-4 (at 125.857 196.596 90) (layer F.SilkS)
     (effects (font (size 1.5 1.5) (thickness 0.3)))
@@
   (gr_line (start 147.9804 81.534) (end 147.9804 233.934) (angle 90) (layer F.Fab) (width 0.2))
   (segment (start 142.2146 204.851) (end 142.1384 204.7748) (width 0.4064) (layer F.Cu) (net 0))
+  (segment (start 128.675 176.149) (end 128.27 176.149) (width 0.4064) (layer F.Cu) (net 1))
+  (segment (start 128.27 176.149) (end 126.492 174.371) (width 0.4064) (layer F.Cu) (net 1))
+  (via (at 126.492 174.371) (size 0.6) (drill 0.4) (layers F.Cu B.Cu) (net 1))
+  (segment (start 137.541 180.721) (end 137.541 178.14) (width 0.4064) (layer F.Cu) (net 2))
+  (segment (start 137.541 178.14) (end 136.947 177.546) (width 0.4064) (layer F.Cu) (net 2))
   (segment (start 140.208 195.707) (end 148.082 195.707) (width 0.4064) (layer B.Cu) (net 2))
   (segment (start 148.082 195.707) (end 149.86 197.485) (width 0.4064) (layer B.Cu) (net 2))
@@
   (segment (start 127.3284 195.326) (end 123.25163 195.326) (width 0.4064) (layer F.Cu) (net 26))
   (segment (start 123.25163 195.326) (end 122.174 195.326) (width 0.4064) (layer F.Cu) (net 26))
+  (segment (start 134.747 177.546) (end 134.597 177.546) (width 0.4064) (layer F.Cu) (net 27))
+  (segment (start 134.597 177.546) (end 133.2 176.149) (width 0.4064) (layer F.Cu) (net 27))
+  (segment (start 133.2 176.149) (end 131.675 176.149) (width 0.4064) (layer F.Cu) (net 27))
   (zone (net 3) (net_name +12V) (layer B.Cu) (hatch edge 0.508)
     (connect_pads yes (clearance 0.254))
