File: DrillBoard-Hardware.kicad_pcb (KiCad board)
At the start: 2 copper layers, 59.7 x 109.8 mm, 190 parts, among them SW1 3P1T_Fused, U1 VNH5019A-E, U10 LS_4, U2 VNH5019A-E, U3 OKI, U4 LS_1, U5 LS_2, U6 TM4C129E_Launchpad_X9, U7 Picoblade-3, U8 Picoblade-3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

Commit message: Modified Gerbers
Other:
- board size 59.7 x 109.8 mm -> 59.7 x 95.5 mm
Changed lines of the file:
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@@
     (links 259)
     (no_connects 0)
-    (area 116.32154 81.433999 179.73926 234.209661)
+    (area 116.32154 81.433999 192.4064 234.209661)
     (thickness 1.6)
-    (drawings 32)
+    (drawings 34)
     (tracks 261)
     (zones 0)
@@
     (47 F.CrtYd user)
     (48 B.Fab user)
-    (49 F.Fab user)
+    (49 F.Fab user hide)
   )
   (setup
@@
     )
   )
+  (gr_line (start 177.6984 186.182) (end 177.6984 141.1224) (layer Edge.Cuts) (width 0.1))
+  (gr_line (start 118.0084 141.0716) (end 118.0084 219.2528) (layer Edge.Cuts) (width 0.1))
+  (gr_line (start 120.4976 138.5824) (end 175.1076 138.5316) (layer Edge.Cuts) (width 0.1))
+  (gr_arc (start 175.1076 141.1224) (end 175.1076 138.5316) (angle 90) (layer Edge.Cuts) (width 0.1))
+  (gr_arc (start 120.4976 141.0716) (end 118.0084 141.0716) (angle 90) (layer Edge.Cuts) (width 0.1))
   (dimension 10.2108 (width 0.3) (layer F.Fab)
     (gr_text "10.211 mm" (at 185.9064 129.3114 270) (layer F.Fab)
@@
   (gr_line (start 175.6156 188.2648) (end 161.1884 188.2648) (layer Edge.Cuts) (width 0.1))
   (gr_arc (start 175.6156 186.182) (end 177.6984 186.182) (angle 90) (layer Edge.Cuts) (width 0.1))
-  (gr_line (start 177.6984 124.1806) (end 177.6984 186.182) (layer Edge.Cuts) (width 0.1))
-  (gr_line (start 118.0084 124.206) (end 177.6984 124.1806) (layer Edge.Cuts) (width 0.1))
-  (gr_line (start 118.0084 219.2528) (end 118.0084 124.206) (layer Edge.Cuts) (width 0.1))
   (gr_text "Drives:\n2 independant motors @ 13A\n1 motor in Parallel @ 26A" (at 175.768 214.249) (layer B.SilkS)
     (effects (font (size 1.5 1.5) (thickness 0.3)) (justify left mirror))

Commit message: Created New Gerb
Other:
- board text added: "Brushed DC Motor Driver, Rev 2 Mars Rover Design Team, 2018 Missouri S&T Andrew Van Horn, Jacob Lipina"
- board text removed: "Brushed DC Motor Driver, Rev 1 Mars Rover Design Team, 2018 Missouri S&T Andrew Van Horn, Jacob Lipina"
Changed lines of the file:
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@@
     (effects (font (size 1.5 1.5) (thickness 0.3)) (justify left mirror))
   )
-  (gr_text "Brushed DC Motor Driver, Rev 1\nMars Rover Design Team, 2018\nMissouri S&T\nAndrew Van Horn, Jacob Lipina\n" (at 139.0904 214.5792) (layer F.SilkS)
+  (gr_text "Brushed DC Motor Driver, Rev 2\nMars Rover Design Team, 2018\nMissouri S&T\nAndrew Van Horn, Jacob Lipina\n" (at 139.0904 214.5792) (layer F.SilkS)
     (effects (font (size 1.5 1.5) (thickness 0.3)))
   )
